File: skye.kicad_pcb (KiCad board)
At the start: 2 copper layers, 13.2 x 24.5 mm, 12 parts, among them IC1 ATTINY85-20SUR, P1 IO, P2 IO, P3 USB_A, U1 WS2812

Commit message: Updated gerber and PDF files, edited silkscreen
Other:
- board text added: "Skye v1"
- board text removed: "Chloé v1"
Changed lines of the file:
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@@
   (gr_arc (start 165.862 88.392) (end 165.862 86.868) (angle 90) (layer Edge.Cuts) (width 0.15))
   (gr_arc (start 166.37 106.426) (end 167.894 106.426) (angle 90) (layer Edge.Cuts) (width 0.15))
-  (gr_text "Chloé v1" (at 161.29 89.662 180) (layer B.Mask)
+  (gr_text "Skye v1" (at 161.29 89.662 180) (layer B.Mask)
     (effects (font (size 1.2 1.2) (thickness 0.2) italic) (justify mirror))
   )
